Commit message: Simulation

File: src/robot_description/urdf/dojo_robot.urdf.xacro (robot description, xacro)
@@ -191,4 +191,46 @@
     <axis xyz="0 1 0"/>
   </joint>
+  <!-- ROS2 Control Hardware Interface -->
+  <ros2_control name="dojo_robot_system" type="system">
+    <hardware>
+      <plugin>gazebo_ros2_control/GazeboSystem</plugin>
+    </hardware>
+    <!-- Front left wheel -->
+    <joint name="front_left_wheel_joint">
+      <command_interface name="velocity">
+        <param name="min">-10</param>
+        <param name="max">10</param>
+      </command_interface>
+      <state_interface name="position"/>
+      <state_interface name="velocity"/>
+    </joint>
+    <!-- Front right wheel -->
+    <joint name="front_right_wheel_joint">
+      <command_interface name="velocity">
+        <param name="min">-10</param>
+        <param name="max">10</param>
+      </command_interface>
+      <state_interface name="position"/>
+      <state_interface name="velocity"/>
+    </joint>
+    <!-- Rear left wheel -->
+    <joint name="rear_left_wheel_joint">
+      <command_interface name="velocity">
+        <param name="min">-10</param>
+        <param name="max">10</param>
+      </command_interface>
+      <state_interface name="position"/>
+      <state_interface name="velocity"/>
+    </joint>
+    <!-- Rear right wheel -->
+    <joint name="rear_right_wheel_joint">
+      <command_interface name="velocity">
+        <param name="min">-10</param>
+        <param name="max">10</param>
+      </command_interface>
+      <state_interface name="position"/>
+      <state_interface name="velocity"/>
+    </joint>
+  </ros2_control>
   <!-- Include Gazebo-specific elements -->
   <xacro:include filename="$(find robot_description)/urdf/dojo_robot.gazebo"/>

Commit message: Simulation

File: src/robot_description/urdf/dojo_robot.urdf.xacro (robot description, xacro)
@@ -166,5 +166,5 @@
     <parent link="base_link"/>
     <child link="camera_link"/>
-    <origin xyz="${base_length/2 - 0.01} 0 ${base_height/2}" rpy="0 0 0"/>
+    <origin xyz="${base_length/2 + 0.01} 0 ${base_height + 0.02}" rpy="0 0 0"/>
   </joint>
   <!-- Wheel joints -->

Commit message: IDK

File: src/robot_description/urdf/dojo_robot.urdf.xacro (robot description, xacro)
@@ -1,6 +1,7 @@
 <?xml version="1.0"?>
 <robot xmlns:xacro="http://www.ros.org/wiki/xacro" name="dojo_robot">
-  <!-- Include common properties -->
+  <!-- Include common properties and sensors -->
   <xacro:include filename="$(find robot_description)/urdf/common_properties.xacro"/>
+  <xacro:include filename="$(find robot_description)/urdf/sensors/rplidar.urdf.xacro"/>
   <!-- Simulation toggle (set by xacro arg) -->
   <xacro:arg name="use_gazebo" default="false"/>
@@ -13,4 +14,13 @@
   <xacro:property name="wheel_separation" value="0.26"/>
   <xacro:property name="wheel_base" value="0.215"/>
+  <!-- Camera parameters -->
+  <xacro:property name="camera_width" value="0.05" />
+  <xacro:property name="camera_height" value="0.03" />
+  <xacro:property name="camera_depth" value="0.05" />
+  <xacro:property name="camera_x" value="0.1" />  <!-- Position in front of the robot -->
+  <xacro:property name="camera_y" value="0.0" />
+  <xacro:property name="camera_z" value="0.05" />
+  <xacro:property name="camera_fps" value="30" />
+  <xacro:property name="camera_hfov" value="1.0472" />  <!-- 60 degrees in radians -->
   <!-- Materials -->
   <material name="dojo_green">

File: src/robot_description/urdf/robot.urdf.xacro (robot description, xacro)
@@ -1,38 +1,38 @@
 <?xml version="1.0"?>
 <robot name="robot_car" xmlns:xacro="http://www.ros.org/wiki/xacro">
-  <!-- Include Gazebo Xacro macros -->
-  <xacro:include filename="$(find gazebo_ros)/launch/empty_world.launch" />
-  <xacro:include filename="$(find gazebo_ros)/launch/helpers/empty_world.launch.py" />
+  <!-- Arguments -->
+  <xacro:arg name="use_ros2_control" default="true" />
   <!-- Include Sensors -->
   <xacro:include filename="$(find robot_description)/urdf/sensors/rplidar.urdf.xacro" />
+  <!-- Camera parameters -->
+  <xacro:property name="camera_width" value="0.05" />
+  <xacro:property name="camera_height" value="0.03" />
+  <xacro:property name="camera_depth" value="0.05" />
+  <xacro:property name="camera_x" value="0.1" />  <!-- Position in front of the robot -->
+  <xacro:property name="camera_y" value="0.0" />
+  <xacro:property name="camera_z" value="0.05" />
+  <xacro:property name="camera_fps" value="30" />
+  <xacro:property name="camera_hfov" value="1.0472" />  <!-- 60 degrees in radians -->
   <!-- Constants -->
   <xacro:property name="PI" value="3.1415926535897931" />
-  <!-- Robot dimensions (in meters) -->
-  <xacro:property name="base_length" value="0.3" />
-  <xacro:property name="base_width" value="0.25" />
-  <xacro:property name="base_height" value="0.15" />
-  <xacro:property name="wheel_radius" value="0.05" />
+  <!-- Robot dimensions (in meters) - Matching dojo_robot.urdf.xacro -->
+  <xacro:property name="base_length" value="0.23" />
+  <xacro:property name="base_width" value="0.28" />
+  <xacro:property name="base_height" value="0.07" />
+  <xacro:property name="wheel_radius" value="0.0325" />
   <xacro:property name="wheel_width" value="0.03" />
-  <xacro:property name="wheel_separation" value="0.3" />
+  <xacro:property name="wheel_separation" value="0.26" />
+  <xacro:property name="wheel_base" value="0.215" />
   <xacro:property name="caster_radius" value="0.01" />
-  <!-- Colors -->
-  <material name="blue">
-    <color rgba="0.0 0.0 0.8 1.0"/>
+  <!-- Materials -->
+  <material name="dojo_green">
+    <color rgba="0.2 0.8 0.2 1"/>
   </material>
-  <material name="black">
-    <color rgba="0.0 0.0 0.0 1.0"/>
+  <material name="wheel_grey">
+    <color rgba="0.4 0.4 0.4 1"/>
   </material>
-  <material name="gray">
-    <color rgba="0.5 0.5 0.5 1.0"/>
-  </material>
-  <!-- Base Link -->
-  <link name="base_footprint">
-    <visual>
-      <origin xyz="0 0 0" rpy="0 0 0"/>
-      <geometry>
-        <box size="0.01 0.01 0.01"/>
-      </geometry>
-    </visual>
-  </link>
+  <!-- Base footprint (for navigation) -->
+  <link name="base_footprint"/>
+  <!-- Base link -->
   <!-- Base -->
   <link name="base_link">
@@ -125,14 +125,71 @@
   <!-- ROS 2 Control -->
   <xacro:if value="$(arg use_ros2_control)">
-    <xacro:include filename="$(find ros2_control_demo_robot)/urdf/diffbot_system.ros2_control.xacro" />
-    <xacro:diffbot_system_robot name="diffbot" prefix="" use_sim="true">
-      <xacro:property name="diff_drive_controller_name" value="diffbot_base_controller" />
-      <xacro:property name="diff_drive_controller_type" value="diff_drive_controller/DiffDriveController" />
-      <xacro:property name="left_wheel_name" value="left_wheel_joint" />
-      <xacro:property name="right_wheel_name" value="right_wheel_joint" />
-      <xacro:property name="wheel_separation" value="${wheel_separation}" />
-      <xacro:property name="wheel_radius" value="${wheel_radius}" />
-    </xacro:diffbot_system_robot>
+    <!-- Gazebo ROS control -->
+    <gazebo>
+      <plugin filename="libgazebo_ros2_control.so" name="gazebo_ros2_control">
+        <parameters>/robot_description</parameters>
+        <controller_manager_node_name>controller_manager</controller_manager_node_name>
+      </plugin>
+    </gazebo>
+    <!-- ROS 2 Control -->
+    <ros2_control name="GazeboSystem" type="system">
+      <hardware>
+        <plugin>gazebo_ros2_control/GazeboSystem</plugin>
+      </hardware>
+      <joint name="left_wheel_joint">
+        <command_interface name="velocity"/>
+        <state_interface name="position"/>
+        <state_interface name="velocity"/>
+      </joint>
+      <joint name="right_wheel_joint">
+        <command_interface name="velocity"/>
+        <state_interface name="position"/>
+        <state_interface name="velocity"/>
+      </joint>
+    </ros2_control>
   </xacro:if>
+  <!-- Camera link -->
+  <link name="camera_link">
+    <visual>
+      <origin xyz="${camera_x} ${camera_y} ${camera_z}" rpy="0 0 0"/>
+      <geometry>
+        <box size="${camera_width} ${camera_height} ${camera_depth}"/>
+      </geometry>
+      <material name="sensor_white"/>
+    </visual>
+    <collision>
+      <origin xyz="${camera_x} ${camera_y} ${camera_z}" rpy="0 0 0"/>
+      <geometry>
+        <box size="${camera_width} ${camera_height} ${camera_depth}"/>
+      </geometry>
+    </collision>
+  </link>
+  <!-- Camera joint -->
+  <joint name="camera_joint" type="fixed">
+    <parent link="base_link"/>
+    <child link="camera_link"/>
+    <origin xyz="0 0 0" rpy="0 0 0"/>
+  </joint>
+  <!-- Camera sensor -->
+  <gazebo reference="camera_link">
+    <sensor type="camera" name="camera1">
+      <update_rate>${camera_fps}</update_rate>
+      <camera name="front">
+        <horizontal_fov>${camera_hfov}</horizontal_fov>
+        <image>
+          <width>640</width>
+          <height>480</height>
+          <format>R8G8B8</format>
+        </image>
+        <clip>
+          <near>0.05</near>
+          <far>100</far>
+        </clip>
+      </camera>
+      <always_on>true</always_on>
+      <update_rate>${camera_fps}</update_rate>
+      <visualize>true</visualize>
+    </sensor>
+  </gazebo>
   <!-- Gazebo plugins -->
   <gazebo>

File: src/robot_description/urdf/sensors/rplidar.urdf.xacro (robot description, xacro)
@@ -4,8 +4,4 @@
   <xacro:property name="lidar_radius" value="0.038" />  <!-- Approximate radius of the LiDAR -->
   <xacro:property name="lidar_height" value="0.045" />   <!-- Approximate height of the LiDAR -->
-  <!-- Position of the LiDAR relative to base_link -->
-  <xacro:property name="lidar_x" value="0.0" />  <!-- Centered front-to-back -->
-  <xacro:property name="lidar_y" value="0.0" />  <!-- Centered left-to-right -->
-  <xacro:property name="lidar_z" value="0.15" />  <!-- On top of the robot -->
   <!-- RPLIDAR A1M8 Link -->
   <link name="laser">
@@ -15,5 +11,5 @@
         <cylinder radius="${lidar_radius}" length="${lidar_height}"/>
       </geometry>
-      <material name="black"/>
+      <material name="sensor_white"/>
     </visual>
     <collision>
@@ -24,9 +20,4 @@
     </collision>
   </link>
-  <!-- Joint from base_link to laser -->
-  <joint name="base_link_to_laser" type="fixed">
-    <parent link="base_link"/>
-    <child link="laser"/>
-    <origin xyz="${lidar_x} ${lidar_y} ${lidar_z}" rpy="0 0 0"/>
-  </joint>
+  <!-- The joint is already defined in dojo_robot.urdf.xacro -->
 </robot>

Commit message: Launch_File Fixes

File: src/robot_description/urdf/dojo_robot.urdf.xacro (robot description, xacro)
@@ -1,4 +1,7 @@
 <?xml version="1.0"?>
 <robot xmlns:xacro="http://www.ros.org/wiki/xacro" name="dojo_robot">
+  <!-- Math constants -->
+  <xacro:property name="M_PI" value="3.1415926535897931" />
+  <xacro:property name="M_PI_2" value="1.5707963267948966" />
   <!-- Include common properties and sensors -->
   <xacro:include filename="$(find robot_description)/urdf/common_properties.xacro"/>
@@ -81,27 +84,4 @@
     </inertial>
   </link>
-  <!-- LiDAR sensor -->
-  <link name="laser">
-    <visual>
-      <geometry>
-        <cylinder radius="0.033" length="0.018"/>
-      </geometry>
-      <origin xyz="0 0 0" rpy="0 0 0"/>
-      <material name="sensor_white"/>
-    </visual>
-    <collision>
-      <geometry>
-        <cylinder radius="0.033" length="0.018"/>
-      </geometry>
-      <origin xyz="0 0 0" rpy="0 0 0"/>
-    </collision>
-    <inertial>
-      <mass value="0.15"/>
-      <origin xyz="0 0 0" rpy="0 0 0"/>
-      <inertia ixx="0.00002" ixy="0.0" ixz="0.0"
-               iyy="0.00002" iyz="0.0"
-               izz="0.00008"/>
-    </inertial>
-  </link>
   <!-- Camera link -->
   <link name="camera_link">
@@ -134,5 +114,5 @@
           <cylinder radius="${wheel_radius}" length="${wheel_width}"/>
         </geometry>
-        <origin xyz="0 0 0" rpy="1.57 0 0"/>
+        <origin xyz="0 0 0" rpy="${reflect * M_PI_2} 0 0"/>
         <material name="wheel_grey"/>
       </visual>
@@ -141,20 +121,74 @@
           <cylinder radius="${wheel_radius}" length="${wheel_width}"/>
         </geometry>
-        <origin xyz="0 0 0" rpy="1.57 0 0"/>
+        <origin xyz="0 0 0" rpy="${reflect * 1.5707963267948966} 0 0"/>
+        <surface>
+          <friction>
+            <ode>
+              <mu>0.8</mu>
+              <mu2>0.8</mu2>
+              <slip1>0.0</slip1>
+              <slip2>0.0</slip2>
+            </ode>
+          </friction>
+        </surface>
       </collision>
       <inertial>
-        <mass value="0.25"/>
-        <origin xyz="0 0 0" rpy="1.57 0 0"/>
-        <inertia ixx="0.0001" ixy="0.0" ixz="0.0"
-                 iyy="0.0003" iyz="0.0"
-                 izz="0.0001"/>
+        <mass value="0.5"/>
+        <inertia ixx="0.0005" ixy="0" ixz="0"
+                 iyy="0.001" iyz="0"
+                 izz="0.0005"/>
       </inertial>
     </link>
   </xacro:macro>
-  <!-- Create all four wheels -->
+  <!-- Create all four wheels with Gazebo properties -->
   <xacro:wheel prefix="front_left" reflect="1"/>
   <xacro:wheel prefix="front_right" reflect="-1"/>
   <xacro:wheel prefix="rear_left" reflect="1"/>
   <xacro:wheel prefix="rear_right" reflect="-1"/>
+  <!-- Gazebo wheel properties -->
+  <gazebo reference="front_left_wheel">
+    <material>Gazebo/Grey</material>
+    <mu1>0.8</mu1>
+    <mu2>0.8</mu2>
+    <kp>1000000.0</kp>
+    <kd>100.0</kd>
+    <fdir1>1 0 0</fdir1>
+    <minDepth>0.001</minDepth>
+    <maxVel>1.0</maxVel>
+    <selfCollide>false</selfCollide>
+  </gazebo>
+  <gazebo reference="front_right_wheel">
+    <material>Gazebo/Grey</material>
+    <mu1>0.8</mu1>
+    <mu2>0.8</mu2>
+    <kp>1000000.0</kp>
+    <kd>100.0</kd>
+    <fdir1>1 0 0</fdir1>
+    <minDepth>0.001</minDepth>
+    <maxVel>1.0</maxVel>
+    <selfCollide>false</selfCollide>
+  </gazebo>
+  <gazebo reference="rear_left_wheel">
+    <material>Gazebo/Grey</material>
+    <mu1>0.8</mu1>
+    <mu2>0.8</mu2>
+    <kp>1000000.0</kp>
+    <kd>100.0</kd>
+    <fdir1>1 0 0</fdir1>
+    <minDepth>0.001</minDepth>
+    <maxVel>1.0</maxVel>
+    <selfCollide>false</selfCollide>
+  </gazebo>
+  <gazebo reference="rear_right_wheel">
+    <material>Gazebo/Grey</material>
+    <mu1>0.8</mu1>
+    <mu2>0.8</mu2>
+    <kp>1000000.0</kp>
+    <kd>100.0</kd>
+    <fdir1>1 0 0</fdir1>
+    <minDepth>0.001</minDepth>
+    <maxVel>1.0</maxVel>
+    <selfCollide>false</selfCollide>
+  </gazebo>
   <!-- Joints -->
   <joint name="base_footprint_joint" type="fixed">
@@ -170,5 +204,5 @@
   <joint name="laser_joint" type="fixed">
     <parent link="sensor_platform"/>
-    <child link="laser"/>
+    <child link="rplidar_link"/>
     <origin xyz="0 0 ${0.038/2 + 0.009}" rpy="0 0 0"/>
   </joint>
@@ -182,24 +216,32 @@
     <parent link="base_link"/>
     <child link="front_left_wheel"/>
-    <origin xyz="${wheel_base/2} ${wheel_separation/2} 0" rpy="0 0 0"/>
+    <origin xyz="${wheel_base/2} ${wheel_separation/2} -${wheel_radius}" rpy="0 0 0"/>
     <axis xyz="0 1 0"/>
+    <limit effort="100" velocity="100"/>
+    <dynamics damping="0.1" friction="0.5"/>
   </joint>
   <joint name="front_right_wheel_joint" type="continuous">
     <parent link="base_link"/>
     <child link="front_right_wheel"/>
-    <origin xyz="${wheel_base/2} ${-wheel_separation/2} 0" rpy="0 0 0"/>
+    <origin xyz="${wheel_base/2} ${-wheel_separation/2} -${wheel_radius}" rpy="0 0 0"/>
     <axis xyz="0 1 0"/>
+    <limit effort="100" velocity="100"/>
+    <dynamics damping="0.1" friction="0.5"/>
   </joint>
   <joint name="rear_left_wheel_joint" type="continuous">
     <parent link="base_link"/>
     <child link="rear_left_wheel"/>
-    <origin xyz="${-wheel_base/2} ${wheel_separation/2} 0" rpy="0 0 0"/>
+    <origin xyz="-${wheel_base/2} ${wheel_separation/2} -${wheel_radius}" rpy="0 0 0"/>
     <axis xyz="0 1 0"/>
+    <limit effort="100" velocity="100"/>
+    <dynamics damping="0.1" friction="0.5"/>
   </joint>
   <joint name="rear_right_wheel_joint" type="continuous">
     <parent link="base_link"/>
     <child link="rear_right_wheel"/>
-    <origin xyz="${-wheel_base/2} ${-wheel_separation/2} 0" rpy="0 0 0"/>
+    <origin xyz="-${wheel_base/2} ${-wheel_separation/2} -${wheel_radius}" rpy="0 0 0"/>
     <axis xyz="0 1 0"/>
+    <limit effort="100" velocity="100"/>
+    <dynamics damping="0.1" friction="0.5"/>
   </joint>
   <!-- ROS2 Control Hardware Interface -->
@@ -207,4 +249,8 @@
     <hardware>
       <plugin>gazebo_ros2_control/GazeboSystem</plugin>
+      <param name="update_rate">100</param>
+      <param name="robot_param">robot_description</param>
+      <param name="robot_param_type">robot_description</param>
+      <param name="use_sim_time">true</param>
     </hardware>
     <!-- Front left wheel -->
@@ -216,4 +262,6 @@
       <state_interface name="position"/>
       <state_interface name="velocity"/>
+      <state_interface name="effort"/>
+      <param name="initial_position">0.0</param>
     </joint>
     <!-- Front right wheel -->
@@ -225,4 +273,6 @@
       <state_interface name="position"/>
       <state_interface name="velocity"/>
+      <state_interface name="effort"/>
+      <param name="initial_position">0.0</param>
     </joint>
     <!-- Rear left wheel -->
@@ -245,7 +295,87 @@
     </joint>
   </ros2_control>
-  <!-- Include Gazebo-specific elements -->
-  <xacro:if value="$(arg use_gazebo)">
-    <xacro:include filename="$(find robot_description)/urdf/dojo_robot.gazebo"/>
-  </xacro:if>
+  <!-- Gazebo properties -->
+  <gazebo>
+    <plugin name="gazebo_ros_control" filename="libgazebo_ros_control.so">
+      <robotNamespace>/</robotNamespace>
+      <robotSimType>gazebo_ros_control/DefaultRobotHWSim</robotSimType>
+    </plugin>
+  </gazebo>
+  <!-- Base link Gazebo properties -->
+  <gazebo reference="base_link">
+    <material>Gazebo/Green</material>
+  </gazebo>
+  <gazebo reference="sensor_platform">
+    <material>Gazebo/Green</material>
+  </gazebo>
+  <gazebo reference="laser">
+    <material>Gazebo/White</material>
+  </gazebo>
+  <gazebo reference="camera_link">
+    <material>Gazebo/White</material>
+  </gazebo>
+  <gazebo reference="front_left_wheel">
+    <material>Gazebo/Grey</material>
+    <mu1>0.8</mu1>
+    <mu2>0.8</mu2>
+    <kp>1000000.0</kp>
+    <kd>100.0</kd>
+  </gazebo>
+  <gazebo reference="front_right_wheel">
+    <material>Gazebo/Grey</material>
+    <mu1>0.8</mu1>
+    <mu2>0.8</mu2>
+    <kp>1000000.0</kp>
+    <kd>100.0</kd>
+  </gazebo>
+  <gazebo reference="rear_left_wheel">
+    <material>Gazebo/Grey</material>
+    <mu1>0.8</mu1>
+    <mu2>0.8</mu2>
+    <kp>1000000.0</kp>
+    <kd>100.0</kd>
+  </gazebo>
+  <gazebo reference="rear_right_wheel">
+    <material>Gazebo/Grey</material>
+    <mu1>0.8</mu1>
+    <mu2>0.8</mu2>
+    <kp>1000000.0</kp>
+    <kd>100.0</kd>
+  </gazebo>
+  <!-- RPLIDAR Gazebo plugin -->
+  <gazebo reference="rplidar_link">
+    <sensor type="ray" name="rplidar">
+      <pose>0 0 0 0 0 0</pose>
+      <visualize>true</visualize>
+      <update_rate>10</update_rate>
+      <ray>
+        <scan>
+          <horizontal>
+            <samples>360</samples>
+            <resolution>1.0</resolution>
+            <min_angle>0.0</min_angle>
+            <max_angle>6.28319</max_angle>
+          </horizontal>
+        </scan>
+        <range>
+          <min>0.15</min>
+          <max>12.0</max>
+          <resolution>0.01</resolution>
+        </range>
+        <noise>
+          <type>gaussian</type>
+          <mean>0.0</mean>
+          <stddev>0.01</stddev>
+        </noise>
+      </ray>
+      <plugin name="gazebo_ros_rplidar_controller" filename="libgazebo_ros_ray_sensor.so">
+        <ros>
+          <namespace>/</namespace>
+          <remapping>~/out:=scan</remapping>
+        </ros>
+        <output_type>sensor_msgs/msg/LaserScan</output_type>
+        <frame_name>rplidar_link</frame_name>
+      </plugin>
+    </sensor>
+  </gazebo>
 </robot>

File: src/robot_description/urdf/robot.urdf.xacro (robot description, xacro)
@@ -5,4 +5,74 @@
   <!-- Include Sensors -->
   <xacro:include filename="$(find robot_description)/urdf/sensors/rplidar.urdf.xacro" />
+  <!-- RPLIDAR Gazebo plugin -->
+  <gazebo reference="rplidar_link">
+    <sensor type="ray" name="rplidar">
+      <pose>0 0 0 0 0 0</pose>
+      <visualize>true</visualize>
+      <update_rate>10</update_rate>
+      <ray>
+        <scan>
+          <horizontal>
+            <samples>360</samples>
+            <resolution>1.0</resolution>
+            <min_angle>0.0</min_angle>
+            <max_angle>6.28319</max_angle>
+          </horizontal>
+        </scan>
+        <range>
+          <min>0.15</min>
+          <max>12.0</max>
+          <resolution>0.01</resolution>
+        </range>
+        <noise>
+          <type>gaussian</type>
+          <mean>0.0</mean>
+          <stddev>0.01</stddev>
+        </noise>
+      </ray>
+      <plugin name="gazebo_ros_rplidar_controller" filename="libgazebo_ros_ray_sensor.so">
+        <ros>
+          <namespace>/</namespace>
+          <remapping>~/out:=scan</remapping>
+        </ros>
+        <output_type>sensor_msgs/msg/LaserScan</output_type>
+        <frame_name>rplidar_link</frame_name>
+      </plugin>
+    </sensor>
+  </gazebo>
+  <!-- Sensor platform for mounting sensors -->
+  <link name="sensor_platform">
+    <visual>
+      <geometry>
+        <box size="0.15 0.085 0.038"/>
+      </geometry>
+      <material name="sensor_white"/>
+    </visual>
+    <collision>
+      <geometry>
+        <box size="0.15 0.085 0.038"/>
+      </geometry>
+    </collision>
+    <inertial>
+      <mass value="0.1"/>
+      <inertia ixx="0.0001" ixy="0" ixz="0" iyy="0.0001" iyz="0" izz="0.0001"/>
+    </inertial>
+  </link>
+  <!-- Joint to connect sensor platform to base -->
+  <joint name="sensor_platform_joint" type="fixed">
+    <parent link="base_link"/>
+    <child link="sensor_platform"/>
+    <origin xyz="0 0 0.05" rpy="0 0 0"/>
+  </joint>
+  <!-- Joint to connect RPLIDAR to sensor platform -->
+  <joint name="laser_joint" type="fixed">
+    <parent link="sensor_platform"/>
+    <child link="rplidar_link"/>
+    <origin xyz="0 0 0.03" rpy="0 0 0"/>
+  </joint>
+  <!-- Materials -->
+  <material name="sensor_white">
+    <color rgba="0.9 0.9 0.9 1"/>
+  </material>
   <!-- Camera parameters -->
   <xacro:property name="camera_width" value="0.05" />

File: src/robot_description/urdf/sensors/rplidar.urdf.xacro (robot description, xacro)
@@ -5,5 +5,5 @@
   <xacro:property name="lidar_height" value="0.045" />   <!-- Approximate height of the LiDAR -->
   <!-- RPLIDAR A1M8 Link -->
-  <link name="laser">
+  <link name="rplidar_link">
     <visual>
       <origin xyz="0 0 ${lidar_height/2}" rpy="0 0 0"/>
